File: STM32F103C8_breakout/STM32F103C8_breakout.kicad_pcb (KiCad board)
At the start: 2 copper layers, 70.8 x 42.5 mm, 26 parts, among them J1 Conn_01x18_Pin, J2 Conn_01x14_Pin, J20 USB-C, J21 Conn_01x02_Pin, U1 STM32F103C8T6, U2 BUCK_REG_3.3V, U3 GPTS203211B, Y1 6 MHz Crystal

Commit message: Finalized PCB Design. Ready for Review.
Parts:
- added R8: 10kΩ, Resistor_SMD:R_0805_2012Metric_Pad1.20x1.40mm_HandSolder, F.Cu at (186.0, 117.0)
Routing:
- net /PB2: track 22.0 -> 31.6 mm
Changed lines of the file:
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@@
 			)
 		)
-		(attr smd dnp)
+		(attr smd)
 		(duplicate_pad_numbers_are_jumpers no)
 		(fp_line
@@
 		)
 	)
+	(footprint "Resistor_SMD:R_0805_2012Metric_Pad1.20x1.40mm_HandSolder"
+		(layer "F.Cu")
+		(at 186 116.975 180)
+		(descr "Resistor SMD 0805 (2012 Metric), square (rectangular) end terminal, IPC-7351 nominal with elongated pad for handsoldering. (Body size source: IPC-SM-782 page 72, https://www.pcb-3d.com/wordpress/wp-content/uploads/ipc-sm-782a_amendment_1_and_2.pdf)")
+		(tags "resistor handsolder")
+		(property "Reference" "R8"
+			(at 0 -1.65 0)
+			(layer "F.SilkS")
+			(effects
+				(font
+					(size 1 1)
+					(thickness 0.15)
+				)
+			)
+		)
+		(property "Value" "10kΩ"
+			(at 0 1.65 0)
+			(layer "F.Fab")
+			(effects
+				(font
+					(size 1 1)
+					(thickness 0.15)
+				)
+			)
+		)
+		(property "Datasheet" ""
+			(at 0 0 0)
+			(layer "F.Fab")
+			(hide yes)
+			(effects
+				(font
+					(size 1.27 1.27)
+				)
+			)
+		)
+		(property "Description" "Resistor, US symbol"
+			(at 0 0 0)
+			(layer "F.Fab")
+			(hide yes)
+			(effects
+				(font
+					(size 1.27 1.27)
+				)
+			)
+		)
+		(property "KiLib_Generator" "SMD_2terminal_chip_molded"
+			(at 0 0 0)
+			(layer "F.SilkS")
+			(hide yes)
+			(effects
+				(font
+					(size 1 1)
+					(thickness 0.15)
+				)
+			)
+		)
+		(property ki_fp_filters "R_*")
+		(sheetname "/")
+		(sheetfile "STM32F103C8_breakout.kicad_sch")
+		(units
+			(unit
+				(name "A")
+				(pins "1" "2")
+			)
+		)
+		(attr smd)
+		(duplicate_pad_numbers_are_jumpers no)
+		(fp_line
+			(start -0.227064 0.735)
+			(end 0.227064 0.735)
+			(stroke
+				(width 0.12)
+				(type solid)
+			)
+			(layer "F.SilkS")
+		)
+		(fp_line
+			(start -0.227064 -0.735)
+			(end 0.227064 -0.735)
+			(stroke
+				(width 0.12)
+				(type solid)
+			)
+			(layer "F.SilkS")
+		)
+		(fp_rect
+			(start -1.85 -0.95)
+			(end 1.85 0.95)
+			(stroke
+				(width 0.05)
+				(type solid)
+			)
+			(fill no)
+			(layer "F.CrtYd")
+		)
+		(fp_rect
+			(start -1 -0.625)
+			(end 1 0.625)
+			(stroke
+				(width 0.1)
+				(type solid)
+			)
+			(fill no)
+			(layer "F.Fab")
+		)
+		(fp_text user "${REFERENCE}"
+			(at 0 0 0)
+			(layer "F.Fab")
+			(effects
+				(font
+					(size 0.5 0.5)
+					(thickness 0.08)
+				)
+			)
+		)
+		(pad "1" smd roundrect
+			(at -1 0 180)
+			(size 1.2 1.4)
+			(layers "F.Cu" "F.Mask" "F.Paste")
+			(roundrect_rratio 0.208333)
+			(net "GNDREF")
+			(pintype "passive")
+		)
+		(pad "2" smd roundrect
+			(at 1 0 180)
+			(size 1.2 1.4)
+			(layers "F.Cu" "F.Mask" "F.Paste")
+			(roundrect_rratio 0.208333)
+			(net "/PB2")
+			(pintype "passive")
+		)
+		(embedded_fonts no)
+		(model "${KICAD10_3DMODEL_DIR}/Resistor_SMD.3dshapes/R_0805_2012Metric.step"
+			(offset
+				(xyz 0 0 0)
+			)
+			(scale
+				(xyz 1 1 1)
+			)
+			(rotate
+				(xyz 0 0 0)
+			)
+		)
+	)
 	(gr_rect
 		(start 126.9 76.65)
@@
 	)
 	(segment
-		(start 156.9 89.551468)
-		(end 156.9 93.232233)
-		(width 0.2)
-		(layer "F.Cu")
-		(net "/JNTRST")
-	)
-	(segment
-		(start 157.451474 88.999994)
-		(end 156.9 89.551468)
-		(width 0.2)
-		(layer "F.Cu")
-		(net "/JNTRST")
-	)
-	(segment
-		(start 156.9 93.232233)
-		(end 157.828177 94.16041)
-		(width 0.2)
-		(layer "F.Cu")
-		(net "/JNTRST")
-	)
-	(segment
-		(start 157.5 88.999994)
-		(end 157.451474 88.999994)
-		(width 0.2)
-		(layer "F.Cu")
-		(net "/JNTRST")
-	)
-	(via
-		(at 157.5 88.999994)
-		(size 0.6)
-		(drill 0.3)
-		(layers "F.Cu" "B.Cu")
-		(net "/JNTRST")
-	)
-	(segment
-		(start 157.5 88.999994)
-		(end 157.5 88.5)
-		(width 0.2)
-		(layer "B.Cu")
-		(net "/JNTRST")
-	)
-	(segment
-		(start 189.82 88.5)
-		(end 190.36 89.04)
-		(width 0.2)
-		(layer "B.Cu")
-		(net "/JNTRST")
-	)
-	(segment
-		(start 157.5 88.5)
-		(end 189.82 88.5)
-		(width 0.2)
-		(layer "B.Cu")
-		(net "/JNTRST")
-	)
-	(segment
 		(start 143.6556 86.107314)
 		(end 143.6556 87.292685)
@@
 	)
 	(segment
+		(start 156.9 89.551468)
+		(end 156.9 93.232233)
+		(width 0.2)
+		(layer "F.Cu")
+		(net "/JNTRST")
+	)
+	(segment
+		(start 157.451474 88.999994)
+		(end 156.9 89.551468)
+		(width 0.2)
+		(layer "F.Cu")
+		(net "/JNTRST")
+	)
+	(segment
+		(start 156.9 93.232233)
+		(end 157.828177 94.16041)
+		(width 0.2)
+		(layer "F.Cu")
+		(net "/JNTRST")
+	)
+	(segment
+		(start 157.5 88.999994)
+		(end 157.451474 88.999994)
+		(width 0.2)
+		(layer "F.Cu")
+		(net "/JNTRST")
+	)
+	(via
+		(at 157.5 88.999994)
+		(size 0.6)
+		(drill 0.3)
+		(layers "F.Cu" "B.Cu")
+		(net "/JNTRST")
+	)
+	(segment
+		(start 157.5 88.999994)
+		(end 157.5 88.5)
+		(width 0.2)
+		(layer "B.Cu")
+		(net "/JNTRST")
+	)
+	(segment
+		(start 189.82 88.5)
+		(end 190.36 89.04)
+		(width 0.2)
+		(layer "B.Cu")
+		(net "/JNTRST")
+	)
+	(segment
+		(start 157.5 88.5)
+		(end 189.82 88.5)
+		(width 0.2)
+		(layer "B.Cu")
+		(net "/JNTRST")
+	)
+	(segment
 		(start 157.548526 89.799997)
 		(end 158.888837 91.140308)
@@
 	)
 	(segment
+		(start 176.4 117)
+		(end 177.55 118.15)
+		(width 0.2)
+		(layer "F.Cu")
+		(net "/PB2")
+	)
+	(segment
 		(start 163.425376 100.425376)
 		(end 163.386036 100.425376)
@@
 	)
 	(segment
+		(start 177.55 118.15)
+		(end 183.825 118.15)
+		(width 0.2)
+		(layer "F.Cu")
+		(net "/PB2")
+	)
+	(segment
 		(start 176.4 113.4)
 		(end 163.425376 100.425376)
 		(width 0.2)
 		(layer "F.Cu")
+		(net "/PB2")
+	)
+	(segment
+		(start 183.825 118.15)
+		(end 185 116.975)
+		(width 0.2)
+		(layer "F.Cu")
